File: blmd_hardware.kicad_pcb (KiCad board)
At the start: 4 copper layers, 50 x 28.5 mm, 88 parts, among them J1 MR30PW-F, J2 control, J3 GND, J4 12V, J5 STLink/V2, J6 STLink-V3, Q1 RH6L040BG, Q2 RH6L040BG, Q3 RH6L040BG, Q4 RH6L040BG, Q5 RH6L040BG, Q6 RH6L040BG, SW1 reset, SW2 SW_DIP_x04, U1 LM5106MMX_NOPB, U10 STM32F303K8T6, U2 LM5106MMX_NOPB, U3 LM5106MMX_NOPB, U4 SI8620BB-B-IS, U5 SI8620BB-B-IS, U6 ACS72981LLRATR-050B3, U7 ACS72981LLRATR-050B3, U8 AP7375(SA), U9 BD41041FJ-C

Commit message: temporary place parts
Parts:
- removed the R10 at (66.7, 36.9)
- removed the R11 at (66.5, 27.7)
- removed the R12 at (67.6, 49.0)
- removed the R13 at (123.8, 54.0)
- removed the R14 at (66.6, 30.4)
- removed the R21 at (105.9, 98.2)
- removed R27: 10k, Resistor_SMD:R_0603_1608Metric_Pad0.98x0.95mm_HandSolder
- removed the R9 at (67.5, 46.6)
- C13, C14, C15, C2, C20, C23, C24, C3, C4, C5, C6, C7, C8, C9, D2, D3, D4, R1, R2: moved to B.Cu
- R10: renamed from R16; moved to B.Cu
- R11: renamed from R17; moved to B.Cu
- R12: renamed from R18; moved to B.Cu
- R13: renamed from R19; moved to B.Cu
- R14: renamed from R20; moved to B.Cu
- R15: renamed from R22; moved to B.Cu
- R16: renamed from R23; moved to B.Cu
- R17: renamed from R24; moved to B.Cu
- R18: renamed from R25; moved to B.Cu
- R9: renamed from R15; moved to B.Cu
- U5: moved to F.Cu
- moved D8 71.4 mm to (83.2, 52.1), turned to -90 degrees
- moved D7 70.3 mm to (81.5, 52.1), turned to -90 degrees
- moved R22 68.6 mm to (83.2, 56.1), turned to 90 degrees
- moved R21 68.1 mm to (81.5, 56.1), turned to 90 degrees
- moved D6 60.3 mm to (79.8, 52.1), turned to -90 degrees
- moved R20 59.0 mm to (79.8, 56.1), turned to 90 degrees
- moved R18 56.0 mm to (94.1, 65.1), turned to -90 degrees
- moved R15 55.9 mm to (99.0, 65.2), turned to 90 degrees
- moved R17 55.9 mm to (95.7, 65.2), turned to 90 degrees
- moved R16 55.9 mm to (97.3, 65.2), turned to 90 degrees
- moved R12 43.7 mm to (89.8, 68.1), turned to -90 degrees
- moved C15 43.4 mm to (82.3, 50.9), turned to 180 degrees
- moved R1 42.4 mm to (77.3, 57.0), turned to 180 degrees
- moved R2 42.4 mm to (77.3, 54.6), turned to 180 degrees
- moved R13 42.4 mm to (88.2, 68.1), turned to -90 degrees
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- renumbered R26 to R19, R28 to R20, R29 to R21, R30 to R22
Connections:
- U5 pad 3: Net-(U5-VIB) -> GNDD
Routing:
- net LOB: track 0.00 -> 6.65 mm
- net LOA: track 0.00 -> 6.65 mm
- net LOC: track 0.00 -> 6.65 mm
- net HOA: track 0.00 -> 2.29 mm
- net HOC: track 0.00 -> 2.29 mm
- net HOB: track 0.00 -> 2.29 mm

Commit message: complete
Parts:
- removed the C14 at (104.5, 61.2)
- removed the C20 at (104.5, 59.3)
- removed J5: STLink/V2, Connector_PinSocket_2.54mm:PinSocket_1x06_P2.54mm_Horizontal
- C19: renamed from C21; value 1u -> 0.047u
- C20: renamed from C22; value 10u -> 0.1u
- SW2: value SW_DIP_x04 -> KHS42E
- U10: value STM32F303K8T6 -> STM32G431KBTx
- U8: value AP7375(SA) -> BD950N1G-C; footprint Package_TO_SOT_SMD:SOT-23-3 -> Package_SO:TSOP-5_1.65x3.05mm_P0.95mm
- moved C21 17.0 mm to (94.6, 64.4)
- moved C22 17.0 mm to (88.8, 63.2), turned to 90 degrees
- moved C20 10.1 mm to (66.3, 55.1), turned to 90 degrees
- moved C17 10.0 mm to (54.8, 69.8)
- moved C13 7.63 mm to (97.1, 52.6), turned to 135 degrees
- moved U8 6.87 mm to (69.0, 55.1), turned to -90 degrees
- moved R23 6.09 mm to (58.8, 69.8), turned to 0 degrees
- moved R19 5.58 mm to (88.2, 52.0)
- moved C14 5.42 mm to (84.3, 55.9), turned to -90 degrees
- moved D5 5.09 mm to (69.0, 58.0), turned to 180 degrees
- moved C19 4.73 mm to (71.7, 55.1), turned to 90 degrees
- moved C10 3.51 mm to (87.1, 63.2)
- moved R18 3.38 mm to (93.9, 68.5), turned to 90 degrees
- moved R16 3.33 mm to (97.3, 68.5)
- moved R17 3.30 mm to (95.6, 68.5)
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- renumbered C15 to C14, C16 to C15, C17 to C16, C18 to C17, C19 to C18, C23 to C21, C24 to C22, R31 to R23, R32 to R24
Connections:
- J6 pad 1: unconnected-(J6-Pin_1-Pad1) -> +3V3
- U10 pad 10: SCA -> ID2
- U10 pad 11: SCC -> SIGA
- U10 pad 12: SIGA -> SIGB
- U10 pad 13: SIGB -> SIGC
- U10 pad 14: SIGC -> GNDD
- U10 pad 15: unconnected-(U10-PB1-Pad15) -> +3V3
- U10 pad 18: SPD1 -> ID3
- U10 pad 19: SPD2 -> ID4
- U10 pad 27: ID1 -> ID_DISP
- U10 pad 28: ID2 -> STATUS
- U10 pad 29: ID3 -> SPD1
- U10 pad 30: ID4 -> SPD2
- U10 pad 5: +3V3 -> SCA
- U10 pad 6: ID_DISP -> SCC
- U10 pad 7: STATUS -> USART_TX
- U10 pad 8: USART_TX -> USART_RX
- U10 pad 9: USART_RX -> ID1
- U6 pad 4: unconnected-(U6-NC-Pad4) -> GNDD
- U6 pad 7: unconnected-(U6-NC-Pad7) -> GNDD
- U7 pad 4: unconnected-(U7-NC-Pad4) -> GNDD
- U8 pad 1: +12V -> unconnected-(U8-NC-Pad1)
- U8 pad 2: +5V -> GND
- U8 pad 3: GND -> unconnected-(U8-NC-Pad3)
Routing:
- net SCA: track 0.00 -> 70.9 mm
- net +5V: track 0.00 -> 56.8 mm, vias 0 -> 3
- net SCC: track 0.00 -> 44.9 mm
- net +5VD: track 0.00 -> 34.9 mm
- net +3V3: track 0.00 -> 34.2 mm, vias 0 -> 6
- net SPD2: track 0.00 -> 30.7 mm, vias 0 -> 1
- net +12V: track 0.00 -> 30.2 mm, vias 0 -> 3
- net HSC: track 0.00 -> 25.8 mm, vias 0 -> 10
- net SPD1: track 0.00 -> 24.4 mm, vias 0 -> 1
- net CANH: track 0.00 -> 23.3 mm
- net CANL: track 0.00 -> 22.3 mm
- net TXD: track 0.00 -> 18.2 mm
- net NRST: track 0.00 -> 17.7 mm, vias 0 -> 1
- net Net-(Q3-G): track 0.00 -> 16.2 mm, vias 0 -> 2
- net USART_TX: track 0.00 -> 16.2 mm, vias 0 -> 1
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- added copper zone on F.Cu, net +12VA
- added copper zone on In1.Cu, net +12VA
- added copper zone on In1.Cu, net +3V3
- added copper zone on B.Cu, net GND
- added copper zone on F.Cu, net GND
- added copper zone on In1.Cu, net GND
- added copper zone on In2.Cu, net GND
- added copper zone on B.Cu, net GNDD
- added copper zone on F.Cu, net GNDD
- added copper zone on In2.Cu, net GNDD
- added copper zone on B.Cu, net GNDPWR
- added copper zone on F.Cu, net GNDPWR
- added copper zone on In1.Cu, net GNDPWR
- added copper zone on In2.Cu, net GNDPWR
- added copper zone on B.Cu, net HSA
- added copper zone on F.Cu, net HSA
- added copper zone on B.Cu, net HSB
- added copper zone on F.Cu, net HSB
- added copper zone on In1.Cu, net HSB
- added copper zone on B.Cu, net HSC
- added copper zone on F.Cu, net HSC
- added copper zone on In1.Cu, net HSC
- added copper zone on B.Cu, net SOA
- added copper zone on F.Cu, net SOA
- added copper zone on In1.Cu, net SOA
- added copper zone on B.Cu, net SOC
- added copper zone on F.Cu, net SOC
- added copper zone on In1.Cu, net SOC
